Commit message: ftsensor topic

File: elfin/elfin_description/urdf/box.urdf.xacro (robot description, xacro)
@@ -1,5 +1,17 @@
 <robot
   name="box" xmlns:xacro="http://www.ros.org/wiki/xacro">
-  <joint name="box_base_joint" type="fixed">
+  <xacro:include filename="$(find elfin_description)/urdf/materials.xacro" />
+  <gazebo reference="box">
+    <visual name='visual'>
+     <material>
+       <script>
+         <uri>file://media/materials/scripts/gazebo.material</uri>
+         <name>Gazebo/Orange</name>
+       </script>
+     </material>
+    </visual>
+  </gazebo>
+  <link name="world"/>
+  <joint name="world_base" type="fixed">
     <origin
       xyz="0 0 0"
@@ -11,4 +23,5 @@
   </joint>
   <link name="box">
+    <static> true </static>
     <visual>
       <origin xyz="0.5 0 0.05" rpy="0 0 0" />
@@ -26,5 +39,5 @@
       <mass value="20" />
       <origin xyz="0 0 0" rpy="0 0 0"/>
-      <inertia ixx="0.01" ixy="0" ixz="0" iyy="0.01" iyz="0" izz="0.01" />
+      <inertia ixx="0.1" ixy="0" ixz="0" iyy="0.1" iyz="0" izz="0.1" />
     </inertial>
   </link>

File: elfin/elfin_description/urdf/elfin3_experiment1.urdf.xacro (robot description, xacro)
@@ -3,6 +3,5 @@
   <xacro:include filename="$(find elfin_description)/urdf/materials.xacro" />
   <xacro:include filename="$(find elfin_description)/urdf/elfin_robot_experiment1.gazebo" />
-  <!-- <xacro:include filename="$(find elfin_description)/urdf/elfin_transmission.xacro" /> -->
-  <xacro:include filename="$(find elfin_description)/urdf/box.urdf.xacro" />
+  <xacro:include filename="$(find elfin_description)/urdf/elfin_transmission.xacro" />
   <xacro:property name="PI" value="3.1415926535897931"/>
   <link name="world"/>
@@ -102,5 +101,5 @@
   <joint
     name="elfin_joint1"
-    type="fixed">
+    type="revolute">
     <origin
       xyz="0 0 0.031"
@@ -160,5 +159,5 @@
   <joint
     name="elfin_joint2"
-    type="fixed">
+    type="revolute">
     <origin
       xyz="-0.068808 0.1615 0"
@@ -218,8 +217,8 @@
   <joint
     name="elfin_joint3"
-    type="fixed">
+    type="revolute">
     <origin
       xyz="0 0.266 0"
-      rpy="${-PI+PI/2} 0 0" />
+      rpy="${-PI} 0 0" />
     <parent
       link="elfin_link2" />
@@ -276,5 +275,5 @@
   <joint
     name="elfin_joint4"
-    type="fixed">
+    type="revolute">
     <origin
       xyz="0.068808 -0.10523 0"
@@ -334,8 +333,8 @@
   <joint
     name="elfin_joint5"
-    type="fixed">
+    type="revolute">
     <origin
       xyz="0 0.21877 0"
-      rpy="${-PI+PI/2} 0 0" />
+      rpy="${-PI} 0 0" />
     <parent
       link="elfin_link4" />
@@ -392,5 +391,5 @@
   <joint
     name="elfin_joint6"
-    type="fixed">
+    type="revolute">
     <origin
       xyz="0 -0.1065 0"
@@ -473,5 +472,5 @@
       <surface>
         <friction>
-          <ode mu="0" mu2="0" slip1="1.0" slip2="1.0" />
+          <ode mu="0.4"/>
         </friction>
       </surface>
