Commit message: adaptive impedance control experiment1

File: elfin/elfin_description/urdf/elfin3_experiment1.urdf.xacro (robot description, xacro)
@@ -435,8 +435,8 @@
     <axis xyz="0 -1 0"/>
     <limit
-      lower="-3.14"
-      upper="3.14"
-      effort="500"
-      velocity="0" />
+      lower="0.0"
+      upper="0.0"
+      effort="0.0"
+      velocity="0.0" />
   </joint>
   <link name="elfin_tool">
@@ -472,5 +472,5 @@
       <surface>
         <friction>
-          <ode mu="0.4"/>
+          <ode mu="0.1"/>
         </friction>
       </surface>

File: elfin/elfin_description/urdf/elfin_transmission.xacro (robot description, xacro)
@@ -56,3 +56,12 @@
       </actuator>
     </transmission>
+    <transmission name="elfin_joint7_trans">
+      <type>transmission_interface/SimpleTransmission</type>
+      <joint name="ft_sensor_joint">
+        <hardwareInterface>hardware_interface/EffortJointInterface</hardwareInterface>
+      </joint>
+      <actuator name="ft_sensor_joint_motor">
+        <mechanicalReduction>1</mechanicalReduction>
+      </actuator>
+    </transmission>
 </robot>

Commit message: add adaptvie torque controller and its models

File: elfin/elfin_description/urdf/elfin3_experiment1.urdf.xacro (robot description, xacro)
@@ -2,6 +2,6 @@
   name="elfin3" xmlns:xacro="http://www.ros.org/wiki/xacro">
   <xacro:include filename="$(find elfin_description)/urdf/materials.xacro" />
-  <xacro:include filename="$(find elfin_description)/urdf/elfin_robot.gazebo" />
-  <xacro:include filename="$(find elfin_description)/urdf/elfin_transmission.xacro" />
+  <xacro:include filename="$(find elfin_description)/urdf/elfin_robot_experiment1.gazebo" />
+  <xacro:include filename="$(find elfin_description)/urdf/elfin_transmission_experiment1.xacro" />
   <xacro:property name="PI" value="3.1415926535897931"/>
   <link name="world"/>
@@ -410,23 +410,81 @@
       velocity="1.57" />
   </joint>
-  <link name="elfin_end_link"/>
-  <joint name="elfin_end_joint" type="fixed">
-    <origin
-      xyz="0 -0.091 0"
-      rpy="${PI/2} ${-PI/2} 0" />
-    <parent
-      link="elfin_link6" />
-    <child
-      link="elfin_end_link" />
-  </joint>
-  <link name="elfin_dummy_gripper"/>
-  <joint name="elfin_dummy_joint" type="fixed">
-    <origin
-      xyz="0 -0.111 0"
-      rpy="${PI/2} ${-PI/2} 0" />
-    <parent
-      link="elfin_link6" />
-    <child
-      link="elfin_dummy_gripper" />
+  <link name="elfin_ft_sensor_link">
+    <collision>
+      <origin xyz="0 0 0" rpy="${PI/2} 0 0"/>
+      <geometry>
+        <cylinder length="0.02" radius="0.04"/>
+      </geometry>
+    </collision>
+    <visual>
+      <origin xyz="0 0 0" rpy="${PI/2} 0 0" />
+      <geometry>
+        <cylinder length="0.02" radius="0.04"/>
+      </geometry>
+    </visual>
+    <inertial>
+      <mass value="0.01" />
+      <origin xyz="0 0 0" rpy="0 0 0"/>
+      <inertia ixx="0.01" ixy="0" ixz="0" iyy="0.01" iyz="0" izz="0.01" />
+    </inertial>
+  </link>
+  <joint name="ft_sensor_joint" type="revolute">
+    <parent link="elfin_link6"/>
+    <child link="elfin_ft_sensor_link"/>
+    <origin xyz="0 -0.08 0" rpy="0 0 0" />
+    <axis xyz="0 -1 0"/>
+    <limit
+      lower="0.0"
+      upper="0.0"
+      effort="0.0"
+      velocity="0.0" />
+  </joint>
+  <link name="elfin_tool">
+    <collision>
+      <origin xyz="0 0 0" rpy="${PI/2} 0 0"/>
+      <geometry>
+        <cylinder length="0.08" radius="0.01"/>
+      </geometry>
+    </collision>
+    <visual>
+      <origin xyz="0 0 0" rpy="${PI/2} 0 0" />
+      <geometry>
+        <cylinder length="0.08" radius="0.01"/>
+      </geometry>
+    </visual>
+    <inertial>
+      <mass value="0.01" />
+      <origin xyz="0 0 0" rpy="0 0 0"/>
+      <inertia ixx="0.01" ixy="0" ixz="0" iyy="0.01" iyz="0" izz="0.01" />
+    </inertial>
+  </link>
+  <joint name="tool_joint" type="fixed">
+    <parent link="elfin_ft_sensor_link"/>
+    <child link="elfin_tool"/>
+    <origin xyz="0 -0.05 0" rpy="0 0 0" />
+  </joint>
+  <link name="elfin_tool_ball">
+    <collision>
+      <origin xyz="0 0 0" rpy="0 0 0"/>
+      <geometry>
+        <sphere radius="0.02"/>
+      </geometry>
+    </collision>
+    <visual>
+      <origin xyz="0 0 0" rpy="0 0 0" />
+      <geometry>
+        <sphere radius="0.02"/>
+      </geometry>
+    </visual>
+    <inertial>
+      <mass value="0.01" />
+      <origin xyz="0 0 0" rpy="0 0 0"/>
+      <inertia ixx="0.01" ixy="0" ixz="0" iyy="0.01" iyz="0" izz="0.01" />
+    </inertial>
+  </link>
+  <joint name="tool_ball_joint" type="fixed">
+    <parent link="elfin_tool"/>
+    <child link="elfin_tool_ball"/>
+    <origin xyz="0 -0.04 0" rpy="0 0 0" />
   </joint>
 </robot>

File: elfin/elfin_description/urdf/elfin3_no_fric_no_joint_limit.urdf.xacro (robot description, xacro)
@@ -2,6 +2,6 @@
   name="elfin3" xmlns:xacro="http://www.ros.org/wiki/xacro">
   <xacro:include filename="$(find elfin_description)/urdf/materials.xacro" />
-  <xacro:include filename="$(find elfin_description)/urdf/elfin_robot.gazebo" />
-  <xacro:include filename="$(find elfin_description)/urdf/elfin_transmission.xacro" />
+  <xacro:include filename="$(find elfin_description)/urdf/elfin_robot_no_fric_no_joint_limit.gazebo" />
+  <xacro:include filename="$(find elfin_description)/urdf/elfin_transmission_no_fric_no_joint_limit.xacro" />
   <xacro:property name="PI" value="3.1415926535897931"/>
   <link name="world"/>
@@ -101,8 +101,8 @@
   <joint
     name="elfin_joint1"
-    type="revolute">
+    type="continuous">
     <origin
       xyz="0 0 0.031"
-      rpy="${PI/2} 0 0" />
+      rpy="${PI/2} 0 ${PI/2}" />
     <parent
       link="elfin_base" />
@@ -112,11 +112,6 @@
       xyz="0 1 0" />
     <dynamics
-      damping="1"
-      friction="1" />
-    <limit
-      lower="-3.14"
-      upper="3.14"
-      effort="120"
-      velocity="1.57" />
+      damping="0"
+      friction="0" />
   </joint>
   <link
@@ -159,5 +154,5 @@
   <joint
     name="elfin_joint2"
-    type="revolute">
+    type="continuous">
     <origin
       xyz="-0.068808 0.1615 0"
@@ -170,11 +165,6 @@
       xyz="-1 0 0" />
     <dynamics
-      damping="1"
-      friction="1" />
-    <limit
-      lower="-2.35"
-      upper="2.35"
-      effort="120"
-      velocity="1.57" />
+      damping="0"
+      friction="0" />
   </joint>
   <link
@@ -217,5 +207,5 @@
   <joint
     name="elfin_joint3"
-    type="revolute">
+    type="continuous">
     <origin
       xyz="0 0.266 0"
@@ -228,11 +218,6 @@
       xyz="1 0 0" />
     <dynamics
-      damping="1"
-      friction="1" />
-    <limit
-      lower="-2.61"
-      upper="2.61"
-      effort="120"
-      velocity="1.57" />
+      damping="0"
+      friction="0" />
   </joint>
   <link
@@ -275,8 +260,8 @@
   <joint
     name="elfin_joint4"
-    type="revolute">
+    type="continuous">
     <origin
       xyz="0.068808 -0.10523 0"
-      rpy="${PI} 0 0" />
+      rpy="${PI/2} 0 0" />
     <parent
       link="elfin_link3" />
@@ -286,11 +271,6 @@
       xyz="0 1 0" />
     <dynamics
-      damping="1"
-      friction="1" />
-    <limit
-      lower="-3.14"
-      upper="3.14"
-      effort="120"
-      velocity="1.57" />
+      damping="0"
+      friction="0" />
   </joint>
   <link
@@ -333,5 +313,5 @@
   <joint
     name="elfin_joint5"
-    type="revolute">
+    type="continuous">
     <origin
       xyz="0 0.21877 0"
@@ -344,11 +324,6 @@
       xyz="1 0 0" />
     <dynamics
-      damping="1"
-      friction="1" />
-    <limit
-      lower="-2.56"
-      upper="2.56"
-      effort="120"
-      velocity="1.57" />
+      damping="0"
+      friction="0" />
   </joint>
   <link
@@ -391,5 +366,5 @@
   <joint
     name="elfin_joint6"
-    type="revolute">
+    type="continuous">
     <origin
       xyz="0 -0.1065 0"
@@ -402,11 +377,6 @@
       xyz="0 -1 0" />
     <dynamics
-      damping="1"
-      friction="1" />
-    <limit
-      lower="-3.14"
-      upper="3.14"
-      effort="120"
-      velocity="1.57" />
+      damping="0"
+      friction="0" />
   </joint>
   <link name="elfin_end_link"/>

File: elfin/elfin_description/urdf/elfin_transmission_experiment_1.xacro (robot description, xacro)
@@ -56,3 +56,12 @@
       </actuator>
     </transmission>
+    <transmission name="elfin_joint7_trans">
+      <type>transmission_interface/SimpleTransmission</type>
+      <joint name="ft_sensor_joint">
+        <hardwareInterface>hardware_interface/EffortJointInterface</hardwareInterface>
+      </joint>
+      <actuator name="ft_sensor_joint_motor">
+        <mechanicalReduction>1</mechanicalReduction>
+      </actuator>
+    </transmission>
 </robot>
