Commit message: sliding mode control, slotine, 1987

File: elfin/elfin_description/urdf/elfin3.urdf.xacro (robot description, xacro)
@@ -402,6 +402,6 @@
       xyz="0 -1 0" />
     <dynamics
-      damping="1"
-      friction="1" />
+      damping="0"
+      friction="100000" />
     <limit
       lower="-3.14"

File: elfin/elfin_description/urdf/elfin3_experiment1.urdf.xacro (robot description, xacro)
@@ -3,5 +3,5 @@
   <xacro:include filename="$(find elfin_description)/urdf/materials.xacro" />
   <xacro:include filename="$(find elfin_description)/urdf/elfin_robot_experiment1.gazebo" />
-  <xacro:include filename="$(find elfin_description)/urdf/elfin_transmission.xacro" />
+  <xacro:include filename="$(find elfin_description)/urdf/elfin_transmission_experiment1.xacro" />
   <xacro:property name="PI" value="3.1415926535897931"/>
   <link name="world"/>

File: elfin/elfin_description/urdf/elfin_transmission.xacro (robot description, xacro)
@@ -56,12 +56,3 @@
       </actuator>
     </transmission>
-    <transmission name="elfin_joint7_trans">
-      <type>transmission_interface/SimpleTransmission</type>
-      <joint name="ft_sensor_joint">
-        <hardwareInterface>hardware_interface/EffortJointInterface</hardwareInterface>
-      </joint>
-      <actuator name="ft_sensor_joint_motor">
-        <mechanicalReduction>1</mechanicalReduction>
-      </actuator>
-    </transmission>
 </robot>

Commit message: Upgrade to ROS 1 Noetic.

File: elfin/elfin_description/urdf/elfin3.urdf.xacro (robot description, xacro)
@@ -1,8 +1,8 @@
 <robot
   name="elfin3" xmlns:xacro="http://www.ros.org/wiki/xacro">
+  <xacro:property name="PI" value="3.1415926535897931"/>
   <xacro:include filename="$(find elfin_description)/urdf/materials.xacro" />
   <xacro:include filename="$(find elfin_description)/urdf/elfin_robot.gazebo" />
   <xacro:include filename="$(find elfin_description)/urdf/elfin_transmission.xacro" />
-  <xacro:property name="PI" value="3.1415926535897931"/>
   <link name="world"/>
   <joint name="world_base" type="fixed">
